Commit message: feature: add right front leg & add material to leg parts

File: www/static/robot.urdf (robot description, URDF)
Before this commit: robot onshape, 9 links, 8 joints
Links:
- link bittle_x_leg: mass 1e-09 -> 0.00320032
- link bittle_x_leg_2: mass 1e-09 -> 0.00320032
- link bittle_x_leg_3: mass 1e-09 -> 0.00320032
- link bittle_x_leg_4: mass 1e-09 -> 0.00320032
- link bittle_x_shank_left: mass 0.014 -> 0.0163164
- link bittle_x_shank_left_2: mass 0.014 -> 0.0163164
- link bittle_x_shank_right: mass 0.014 -> 0.0163164
- link bittle_x_shank_right_2: mass 0.014 -> 0.0163164

Commit message: feature: add floot & collision spheres

File: www/static/robot.urdf (robot description, URDF)
Before this commit: robot onshape, 9 links, 8 joints
Links:
- added link left_back_foot, mass 1e-9
- added link left_front_foot, mass 1e-9
- added link right_back_foot, mass 1e-9
- added link right_front_foot, mass 1e-9
Joints:
- added joint left_back_foot_frame: type fixed, parent bittle_x_shank_left_2, child left_back_foot, origin xyz=-0.048 2.08167e-17 -0.0165 rpy=-3.14159 1.84363e-30 -2.66751e-29, axis 0 0 0
- added joint left_front_foot_frame: type fixed, parent bittle_x_shank_left, child left_front_foot, origin xyz=-0.048 -6.93889e-18 -0.0165 rpy=3.14159 1.37705e-30 9.06996e-29, axis 0 0 0
- added joint right_back_foot_frame: type fixed, parent bittle_x_shank_right_2, child right_back_foot, origin xyz=-0.048 6.93889e-18 -0.0165 rpy=4.80984e-18 2.77556e-16 -6.93889e-17, axis 0 0 0
- added joint right_front_foot_frame: type fixed, parent bittle_x_shank_right, child right_front_foot, origin xyz=-0.048 1.38778e-17 -0.0165 rpy=2.39147e-18 2.77556e-16 -6.93889e-17, axis 0 0 0

Commit message: feature: add knee collision points

File: www/static/robot.urdf (robot description, URDF)
Before this commit: robot onshape, 13 links, 12 joints
Links:
- added link left_back_knee, mass 1e-9
- added link left_front_knee, mass 1e-9
- added link right_back_knee, mass 1e-9
- added link right_front_knee, mass 1e-9
Joints:
- added joint left_back_knee_frame: type fixed, parent bittle_x_leg_4, child left_back_knee, origin xyz=-0.0554318 3.16941e-13 -0.0041 rpy=1.5708 7.96211e-18 5.36897e-12, axis 0 0 0
- added joint left_front_knee_frame: type fixed, parent bittle_x_leg, child left_front_knee, origin xyz=-0.0554318 3.16941e-13 -0.0041 rpy=1.5708 -1.88644e-17 5.36902e-12, axis 0 0 0
- added joint right_back_knee_frame: type fixed, parent bittle_x_leg_3, child right_back_knee, origin xyz=-0.0554318 3.16913e-13 -0.0041 rpy=1.5708 1.33352e-17 5.36902e-12, axis 0 0 0
- added joint right_front_knee_frame: type fixed, parent bittle_x_leg_2, child right_front_knee, origin xyz=-0.0554318 3.16934e-13 -0.0041 rpy=1.5708 -5.05038e-18 5.36902e-12, axis 0 0 0

Commit message: feature: add cover

File: www/static/robot.urdf (robot description, URDF)
Before this commit: robot onshape, 17 links, 16 joints
Links:
- link chassis: mass 0.0632774 -> 0.0726024; geometry visual mesh filename=package://assets/chassis.stl; visual mesh filename=package://assets/cover.stl

Commit message: feature: add head joint & more body parts

File: www/static/robot.urdf (robot description, URDF)
Before this commit: robot onshape, 17 links, 16 joints
Links:
- added link bittle_x_head, mass 0.022581; visual mesh filename=package://assets/head_1.stl; visual mesh filename=package://assets/head_2.stl
- link chassis: mass 0.0726024 -> 0.147477; geometry visual mesh filename=package://assets/809_25_v1.stl; visual mesh filename=package://assets/battcase.stl
Joints:
- added joint head: type revolute, parent chassis, child bittle_x_head, origin xyz=-0.00626294 -0.0435043 0.01074 rpy=3.14159 -0.523599 1.5708, axis 0 0 1, limit lower=-3.141592653589793 upper=3.141592653589793 effort=10 velocity=10
- joint left_back: origin xyz=0.0422987 0.0548412 0.000213389 rpy=-3.14159 -1.53589 3.14159 -> xyz=0.0422033 0.0548412 -0.000503935 rpy=1.68824e-17 -1.5708 0
- joint left_back_foot_frame: origin xyz=-0.048 2.08167e-17 -0.0165 rpy=-3.14159 1.84363e-30 -2.66751e-29 -> xyz=-0.048 0 -0.0165 rpy=-3.14159 -1.56548e-30 -1.34966e-29
- joint left_back_knee: origin xyz=-0.046 3.68643e-13 -0.00215 rpy=-3.14159 2.24001e-16 1.5708 -> xyz=-0.046 3.68636e-13 -0.00215 rpy=-3.14159 2.24001e-16 1.5708
- joint left_back_knee_frame: origin xyz=-0.0554318 3.16941e-13 -0.0041 rpy=1.5708 7.96211e-18 5.36897e-12 -> xyz=-0.0554318 3.16934e-13 -0.0041 rpy=1.5708 -2.65902e-28 5.36897e-12
- joint left_front: origin xyz=0.0422987 -0.0501588 0.000213389 rpy=-3.14159 -1.53589 3.14159 -> xyz=0.0422033 -0.0501588 -0.000503935 rpy=1.08732e-17 -1.5708 0
- joint left_front_foot_frame: origin xyz=-0.048 -6.93889e-18 -0.0165 rpy=3.14159 1.37705e-30 9.06996e-29 -> xyz=-0.048 6.93889e-18 -0.0165 rpy=3.14159 -1.14548e-30 -4.49613e-30
- joint left_front_knee: origin xyz=-0.046 3.68636e-13 -0.00215 rpy=-3.14159 2.77413e-16 1.5708 -> xyz=-0.046 3.68629e-13 -0.00215 rpy=-3.14159 2.77413e-16 1.5708
- joint left_front_knee_frame: origin xyz=-0.0554318 3.16941e-13 -0.0041 rpy=1.5708 -1.88644e-17 5.36902e-12 -> xyz=-0.0554318 3.16934e-13 -0.0041 rpy=1.5708 -1.38778e-17 5.36902e-12
- joint right_back: origin xyz=-0.0548246 0.0548119 0.000213389 rpy=3.14159 -1.53589 2.18867e-11 -> xyz=-0.0547292 0.0548119 -0.000503935 rpy=-3.14159 -1.5708 0
- joint right_back_foot_frame: origin xyz=-0.048 6.93889e-18 -0.0165 rpy=4.80984e-18 2.77556e-16 -6.93889e-17 -> xyz=-0.048 6.93889e-18 -0.0165 rpy=9.24446e-33 2.77556e-16 -6.93889e-17
- joint right_back_knee: origin xyz=-0.046 3.68643e-13 -0.00215 rpy=3.14159 -2.74609e-16 -1.5708 -> xyz=-0.046 3.6865e-13 -0.00215 rpy=-3.14159 -2.74609e-16 -1.5708
- joint right_back_knee_frame: origin xyz=-0.0554318 3.16913e-13 -0.0041 rpy=1.5708 1.33352e-17 5.36902e-12 -> xyz=-0.0554318 3.1692e-13 -0.0041 rpy=1.5708 6.93889e-18 5.36902e-12
- joint right_front: origin xyz=-0.0548246 -0.0501881 0.000213389 rpy=3.14159 -1.53589 2.19137e-11 -> xyz=-0.0547292 -0.0501881 -0.000503935 rpy=-3.14159 -1.5708 0
- joint right_front_foot_frame: origin xyz=-0.048 1.38778e-17 -0.0165 rpy=2.39147e-18 2.77556e-16 -6.93889e-17 -> xyz=-0.048 6.93889e-18 -0.0165 rpy=7.70372e-33 2.77556e-16 -6.93889e-17
- joint right_front_knee: origin xyz=-0.046 3.68691e-13 -0.00215 rpy=-3.14159 -2.80217e-16 -1.5708 -> xyz=-0.046 3.68677e-13 -0.00215 rpy=3.14159 -2.80217e-16 -1.5708
- joint right_front_knee_frame: origin xyz=-0.0554318 3.16934e-13 -0.0041 rpy=1.5708 -5.05038e-18 5.36902e-12 -> xyz=-0.0554318 3.16934e-13 -0.0041 rpy=1.5708 -3.01693e-29 5.36902e-12
