Commit message: feat: add more collision geom & add joint friction

File: docs/robot.urdf (robot description, URDF)
Before this commit: robot onshape, 18 links, 17 joints
Links:
- added link head, mass 1e-9
- added link left_back_shoulder, mass 1e-9
- added link left_front_shoulder, mass 1e-9
- added link right_back_shoulder, mass 1e-9
- added link right_front_shoulder, mass 1e-9
- added link tail, mass 1e-9
- link bittle_x_leg: geometry visual mesh filename=package://assets/809_25_v1.stl; visual mesh filename=package://assets/809_25_v1.stl
- link bittle_x_leg_2: geometry visual mesh filename=package://assets/809_25_v1.stl; visual mesh filename=package://assets/809_25_v1.stl
- link bittle_x_leg_3: geometry visual mesh filename=package://assets/809_25_v1.stl; visual mesh filename=package://assets/809_25_v1.stl
- link bittle_x_leg_4: geometry visual mesh filename=package://assets/809_25_v1.stl; visual mesh filename=package://assets/809_25_v1.stl
- link chassis: mass 0.147477 -> 0.158971
Joints:
- added joint head_frame: type fixed, parent bittle_x_head, child head, origin xyz=-0.00456954 -0.00012664 -0.0434696 rpy=-2.74378 7.34748e-32 -1.5708, axis 0 0 0
- added joint left_back_shoulder_frame: type fixed, parent chassis, child left_back_shoulder, origin xyz=0.0347033 0.0548412 -0.000503935 rpy=1.5708 0.523599 1.5708, axis 0 0 0
- added joint left_front_shoulder_frame: type fixed, parent chassis, child left_front_shoulder, origin xyz=0.0347033 -0.0501588 -0.000503935 rpy=-1.5708 0.523599 -1.5708, axis 0 0 0
- added joint right_back_shoulder_frame: type fixed, parent chassis, child right_back_shoulder, origin xyz=-0.0472292 0.0548119 -0.000503935 rpy=-1.5708 0.523599 1.5708, axis 0 0 0
- added joint right_front_shoulder_frame: type fixed, parent chassis, child right_front_shoulder, origin xyz=-0.0472292 -0.0501881 -0.000503935 rpy=1.5708 0.523599 -1.5708, axis 0 0 0
- added joint tail_frame: type fixed, parent chassis, child tail, origin xyz=-0.00639673 0.085276 0.0444891 rpy=-7.64786e-13 -3.43475e-16 -5.96644e-17, axis 0 0 0
